File: board/misteryshield20k_rpipico/MiSTeryShield20kRPiPico.kicad_pcb (KiCad board)
At the start: 2 copper layers, 100 x 57 mm, 57 parts, among them J1 Joystick, J10 Conn_02x04_Pin, J11 USB_A_Stacked, J12 USB_A_Stacked, J2 DS2, J3 Conn_02x04_Pin, J4 Conn_01x20_Pin, J5 MIDI IN, J6 MIDI OUT, J7 Conn_01x20_Pin, J8 Conn_01x20_Pin, J9 Conn_01x20_Pin, Q1 BSS123, Q2 BSS123, Q3 BSS123, Q4 BSS123, Q5 BSS123, Q6 BSS123, U1 H11L1S, U2 74LVC2G14, U4 CH334U, Y1 Crystal_GND24

Commit message: MiSTeryShield20kRPiPico_V2
Parts:
- turned J2 to 0 degrees
Routing:
- net P73: track 138.6 -> 158.2 mm, vias 2 -> 3
- net P31: track 116.3 -> 126.6 mm, vias 4 -> 6
- net GND: track 22.1 -> 28.6 mm, vias 284 -> 285
- net P74: track 125.5 -> 123.2 mm, vias 4 -> 5
- net +3.3V: track 254.7 -> 252.5 mm
- net +5V: track 305.8 -> 304.5 mm
- net P77: track 122.5 -> 123.7 mm, vias 2 -> 3
Other:
- board text added: "Rev. V2"
