File: board/misteryshield20k_rpipico/MiSTeryShield20kRPiPico_usbhub.kicad_sch (KiCad schematic)
At the start: 18 parts, among them J10 Conn_02x04_Pin, J11 USB_A_Stacked, J12 USB_A_Stacked, J8 Conn_01x20_Pin, J9 Conn_01x20_Pin, U4 CH334U, Y1 Crystal_GND24

Commit message: add updated shield (DS2 removed)
Parts:
- removed A1: Raspberry_Pi_Pico_W, misteryshield20kpico:Raspberry_Pi_Pico_W, symbol MiSTeryShield20kRPiPico:Raspberry_Pi_Pico_W
- removed C4, C7: 1uF, Capacitor_SMD:C_0805_2012Metric, symbol Device:C_Small
- removed C5: 10uF, Capacitor_SMD:C_0805_2012Metric, symbol Device:C_Small
- removed C6: 100nF, Capacitor_SMD:C_0805_2012Metric, symbol Device:C_Small
- removed D2, D3, D4: green, LED_SMD:LED_0805_2012Metric, symbol Device:LED
- removed J10: Conn_02x04_Pin, Connector_PinHeader_2.54mm:PinHeader_2x04_P2.54mm_Vertical, symbol Connector:Conn_01x08_Pin
- removed J11, J12: USB_A_Stacked, MiSTeryShield20kRPiPico:USB_A_Wuerth_61400826021_Horizontal_Stacked, symbol misteryshield20kpico:USB_A_Stacked
- removed J8, J9: Conn_01x20_Pin, Connector_PinSocket_2.54mm:PinSocket_1x20_P2.54mm_Vertical, symbol Connector:Conn_01x20_Pin
- removed R18, R19, R20: 560, Resistor_SMD:R_0805_2012Metric, symbol Device:R
- removed U4: CH334U, Package_SO:SSOP-28_3.9x9.9mm_P0.635mm, symbol wch_mcu_peripheral:CH334U
- removed Y1: Crystal_GND24, Crystal:Crystal_SMD_3225-4Pin_3.2x2.5mm, symbol Device:Crystal_GND24
Connections:
- no-connect marks 26 -> 0
Other:
- company: Stefan Voss -> (none)
- title: MiSTeryShield20KRPiPico -> (none)
