File: board/misteryshield20k_rpipico/MiSTeryShield20kRPiPicoUSB.kicad_pcb (KiCad board)
At the start: 2 copper layers, 100 x 57 mm, 56 parts, among them J1 Joystick, J10 Conn_02x04_Pin, J11 USB_A_Stacked, J12 USB_A_Stacked, J3 Conn_02x04_Pin, J4 Conn_01x20_Pin, J5 MIDI IN, J6 MIDI OUT, J7 Conn_01x20_Pin, J8 Conn_01x20_Pin, J9 Conn_01x20_Pin, Q1 2N7002, Q2 2N7002, Q3 2N7002, Q4 2N7002, Q5 2N7002, Q6 2N7002, U1 H11L1S, U2 74LVC2G14, U4 CH334U, Y1 Crystal_GND24

Commit message: board update
Connections:
- J5 pad 4: Net-(D1-A) -> Net-(J5-Pad4)
- J5 pad 5: Net-(J5-Pad5) -> Net-(D1-A)
- R15 pad 1: Net-(J5-Pad5) -> Net-(J5-Pad4)
Routing:
- net Net-(J5-Pad5): track 90.7 -> 0.00 mm, vias 1 -> 0
- net Net-(J5-Pad4): track 0.00 -> 80.0 mm, vias 0 -> 1
- net Net-(D1-A): track 83.7 -> 96.7 mm
Other:
- board text added: "Rev. V3"
- board text removed: "Rev. V1"
