File: board/misteryshield20k_rpipico/MiSTeryShield20kRPiPicoUSB.kicad_sch (KiCad schematic)
At the start: 40 parts, among them J1 Joystick, J3 Conn_02x04_Pin, J4 Conn_01x20_Pin, J5 MIDI IN, J6 MIDI OUT, J7 Conn_01x20_Pin, Q1 2N7002, Q2 2N7002, Q3 2N7002, Q4 2N7002, Q5 2N7002, Q6 2N7002, U1 H11L1S, U2 74LVC2G14

Commit message: board update
Connections:
- net at D1.2 (A), U1.2: now also J5.5; no longer J5.4
- net at R15.1: now also J5.4; no longer J5.5
Other:
- moved on the sheet: J5
Changed lines of the file:
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@@
 (kicad_sch
-	(version 20231120)
+	(version 20250114)
 	(generator "eeschema")
-	(generator_version "8.0")
+	(generator_version "9.0")
 	(paper "A4")
 	(title_block
 		(title "MiSTeryShield20KPiPico")
-		(date "2025-01-30")
-		(rev "V1")
+		(date "2025-08-09")
+		(rev "V3")
 		(company "Stefan Voss")
 		(comment 3 "(c) 2025 by Stefan Voss")
 		(comment 4 "MiSTery Pi Pico WLAN Shield for Tang Nano 20K")
 	)
+	(text "6 * Levelshifter 5V/3.3V"
+		(exclude_from_sim no)
+		(at 85.09 89.535 0)
+		(effects
+			(font
+				(size 1.27 1.27)
+			)
+			(justify left bottom)
+		)
+	)
+	(text "Spare IO"
+		(exclude_from_sim no)
+		(at 92.075 156.845 0)
+		(effects
+			(font
+				(size 1.27 1.27)
+			)
+			(justify left bottom)
+		)
+	)
+	(text "Place near U1"
+		(exclude_from_sim no)
+		(at 27.432 188.214 0)
+		(effects
+			(font
+				(size 1.27 1.27)
+			)
+		)
+	)
+	(text "6 * 10K"
+		(exclude_from_sim no)
+		(at 57.15 45.72 0)
+		(effects
+			(font
+				(size 1.27 1.27)
+			)
+			(justify left bottom)
+		)
+	)
+	(text "6 x 2N7002"
+		(exclude_from_sim no)
+		(at 76.2 52.705 0)
+		(effects
+			(font
+				(size 1.27 1.27)
+			)
+			(justify left bottom)
+		)
+	)
+	(text "6 * 10K"
+		(exclude_from_sim no)
+		(at 105.41 46.355 0)
+		(effects
+			(font
+				(size 1.27 1.27)
+			)
+			(justify left bottom)
+		)
+	)
 	(junction
 		(at 107.95 69.85)
@@
 	)
 	(no_connect
-		(at 163.83 116.84)
+		(at 185.42 116.84)
 	)
 	(no_connect
@@
 	)
 	(no_connect
-		(at 171.45 124.46)
+		(at 177.8 124.46)
 	)
 	(no_connect
@@
 	)
 	(no_connect
-		(at 179.07 116.84)
+		(at 170.18 116.84)
 	)
 	(wire
@@
 	(wire
 		(pts
-			(xy 179.07 121.92) (xy 179.07 124.46)
-		)
-		(stroke
-			(width 0)
-			(type default)
-		)
-	)
-	(wire
-		(pts
 			(xy 100.33 74.93) (xy 149.86 74.93)
 		)
@@
 	(wire
 		(pts
+			(xy 170.18 121.92) (xy 170.18 124.46)
+		)
+		(stroke
+			(width 0)
+			(type default)
+		)
+	)
+	(wire
+		(pts
 			(xy 104.14 72.39) (xy 104.14 78.105)
 		)
@@
 	(wire
 		(pts
-			(xy 107.95 69.85) (xy 149.86 69.85)
+			(xy 185.42 119.38) (xy 190.5 119.38)
 		)
 		(stroke
@@
 	(wire
 		(pts
-			(xy 199.39 57.15) (xy 242.57 57.15)
+			(xy 107.95 69.85) (xy 149.86 69.85)
 		)
 		(stroke
@@
 	(wire
 		(pts
-			(xy 179.07 119.38) (xy 190.5 119.38)
+			(xy 199.39 57.15) (xy 242.57 57.15)
 		)
 		(stroke
@@
 	(wire
 		(pts
-			(xy 162.56 119.38) (xy 163.83 119.38)
-		)
-		(stroke
-			(width 0)
-			(type default)
-		)
-	)
-	(wire
-		(pts
 			(xy 199.39 49.53) (xy 242.57 49.53)
 		)
@@
 	(wire
 		(pts
+			(xy 162.56 119.38) (xy 170.18 119.38)
+		)
+		(stroke
+			(width 0)
+			(type default)
+		)
+	)
+	(wire
+		(pts
 			(xy 199.39 59.69) (xy 242.57 59.69)
 		)
@@
 		)
 	)
-	(text "6 * Levelshifter 5V/3.3V"
-		(exclude_from_sim no)
-		(at 85.09 89.535 0)
-		(effects
-			(font
-				(size 1.27 1.27)
-			)
-			(justify left bottom)
-		)
-	)
-	(text "Spare IO"
-		(exclude_from_sim no)
-		(at 92.075 156.845 0)
-		(effects
-			(font
-				(size 1.27 1.27)
-			)
-			(justify left bottom)
-		)
-	)
-	(text "Place near U1"
-		(exclude_from_sim no)
-		(at 27.432 188.214 0)
-		(effects
-			(font
-				(size 1.27 1.27)
-			)
-		)
-	)
-	(text "6 * 10K"
-		(exclude_from_sim no)
-		(at 57.15 45.72 0)
-		(effects
-			(font
-				(size 1.27 1.27)
-			)
-			(justify left bottom)
-		)
-	)
-	(text "6 x 2N7002"
-		(exclude_from_sim no)
-		(at 76.2 52.705 0)
-		(effects
-			(font
-				(size 1.27 1.27)
-			)
-			(justify left bottom)
-		)
-	)
-	(text "6 * 10K"
-		(exclude_from_sim no)
-		(at 105.41 46.355 0)
-		(effects
-			(font
-				(size 1.27 1.27)
-			)
-			(justify left bottom)
-		)
-	)
 	(label "IO_LEFT"
 		(at 135.89 72.39 0)
-		(fields_autoplaced yes)
 		(effects
 			(font
@@
 	(label "BTN2"
 		(at 41.275 64.77 0)
-		(fields_autoplaced yes)
 		(effects
 			(font
@@
 	(label "LEFT"
 		(at 41.275 72.39 0)
-		(fields_autoplaced yes)
 		(effects
 			(font
@@
 	(label "UP"
 		(at 41.275 82.55 0)
-		(fields_autoplaced yes)
 		(effects
 			(font
@@
 	(label "BTN1"
 		(at 41.275 80.01 0)
-		(fields_autoplaced yes)
 		(effects
 			(font
@@
 	(label "IO_BTN1"
 		(at 135.89 62.23 0)
-		(fields_autoplaced yes)
 		(effects
 			(font
@@
 	(label "IO_UP"
 		(at 135.89 67.31 0)
-		(fields_autoplaced yes)
 		(effects
 			(font
@@
 	(label "IO_DOWN"
 		(at 135.89 64.77 0)
-		(fields_autoplaced yes)
 		(effects
 			(font
@@
 	(label "IO_BTN2"
 		(at 135.89 74.93 0)
-		(fields_autoplaced yes)
 		(effects
 			(font
@@
 	(label "IO_RIGHT"
 		(at 135.89 69.85 0)
-		(fields_autoplaced yes)
 		(effects
 			(font
@@
 	(label "DOWN"
 		(at 41.275 77.47 0)
-		(fields_autoplaced yes)
 		(effects
 			(font
@@
 	(label "RIGHT"
 		(at 41.275 67.31 0)
-		(fields_autoplaced yes)
 		(effects
 			(font
@@
 		(dnp no)
 		(property "Reference" "D1"
-			(at 158.75 122.555 90)
+			(at 156.464 125.984 90)
 			(effects
 				(font
@@
 		)
 		(property "Value" "1N4148W"
-			(at 165.1 124.46 90)
+			(at 162.814 127.762 90)
 			(effects
 				(font
@@
 	(symbol
 		(lib_id "power:GND")
-		(at 179.07 124.46 0)
+		(at 170.18 124.46 0)
 		(unit 1)
 		(exclude_from_sim no)
@@
 		(dnp no)
 		(property "Reference" "#PWR053"
-			(at 179.07 130.81 0)
+			(at 170.18 130.81 0)
 			(effects
 				(font
@@
 		)
 		(property "Value" "GND"
-			(at 180.975 128.27 0)
+			(at 172.085 128.27 0)
 			(effects
 				(font
@@
 		)
 		(property "Footprint" ""
-			(at 179.07 124.46 0)
+			(at 170.18 124.46 0)
 			(effects
 				(font
@@
 		)
 		(property "Datasheet" ""
-			(at 179.07 124.46 0)
+			(at 170.18 124.46 0)
 			(effects
 				(font
@@
 		)
 		(property "Description" ""
-			(at 179.07 124.46 0)
+			(at 170.18 124.46 0)
 			(effects
 				(font
@@
 	(symbol
 		(lib_id "misteryshield20kpico:DIN-5_180degree")
-		(at 171.45 116.84 180)
+		(at 177.8 116.84 0)
+		(mirror x)
 		(unit 1)
 		(exclude_from_sim no)
@@
 		(dnp no)
 		(property "Reference" "J5"
-			(at 169.672 107.696 0)
+			(at 179.578 107.696 0)
 			(effects
 				(font
@@
 		)
 		(property "Value" "MIDI IN"
-			(at 171.45 109.728 0)
+			(at 177.8 109.728 0)
 			(effects
 				(font
@@
 		)
 		(property "Footprint" "MiSTeryShield20kRPiPico:DIN-5_180degree"
-			(at 171.45 116.84 0)
+			(at 177.8 116.84 0)
 			(effects
 				(font
@@
 		)
 		(property "Datasheet" "http://www.mouser.com/ds/2/18/40_c091_abd_e-75918.pdf"
-			(at 171.45 116.84 0)
+			(at 177.8 116.84 0)
 			(effects
 				(font
@@
 		)
 		(property "Description" "5-pin DIN connector (5-pin DIN-5 stereo)"
-			(at 171.45 116.84 0)
+			(at 177.8 116.84 0)
 			(effects
 				(font
@@
 		)
 		(property "LCSC Part #" "C2939346"
-			(at 171.45 116.84 0)
+			(at 177.8 116.84 0)
 			(effects
 				(font
@@
 		)
 		(property "JLCPCB Position Offset" ""
-			(at 171.45 116.84 0)
+			(at 177.8 116.84 0)
 			(effects
 				(font
@@
 		)
 		(property "JLCPCB Rotation Offset" ""
-			(at 171.45 116.84 0)
+			(at 177.8 116.84 0)
 			(effects
 				(font
@@
 		)
 		(property "Comment" "DIN-5_180degree"
-			(at 171.45 116.84 0)
+			(at 177.8 116.84 0)
 			(effects
 				(font
@@
 		(at 242.57 43.688)
 		(size 27.94 27.178)
+		(exclude_from_sim no)
+		(in_bom yes)
+		(on_board yes)
+		(dnp no)
 		(stroke
 			(width 0.1524)
@@
 		)
 	)
+	(embedded_fonts no)
 )
